File: USB-to-TTL Serial UART Converter.kicad_pcb (KiCad board)
At the start: 2 copper layers, 12 parts, among them J1 USB_C_Receptacle, J2 Conn_01x06_Pin, U1 CH340G, Y1 Crystal_GND2

Commit message: Add files via upload
Parts:
- moved R1 127.4 mm to (48.6, 126.5), turned to -90 degrees
- moved D1 125.1 mm to (38.8, 118.5), turned to -90 degrees
- moved J1 96.7 mm to (74.1, 133.1), turned to 0 degrees
- moved C3 96.7 mm to (47.6, 116.8), turned to -90 degrees
- moved R3 80.6 mm to (86.4, 137.1), turned to -90 degrees
- moved R2 76.6 mm to (86.6, 127.1)
- moved J2 70.6 mm to (58.2, 118.8), turned to 180 degrees
- moved C1 68.6 mm to (70.0, 109.0), turned to -90 degrees
- moved U1 54.2 mm to (72.4, 96.6), turned to 90 degrees
- moved C2 50.2 mm to (78.8, 109.2), turned to -90 degrees
- moved Y1 50.2 mm to (74.6, 83.6), turned to 180 degrees
- moved C4 44.5 mm to (86.8, 109.0)
Routing:
- net GND: track 4.41 -> 242.6 mm, vias 0 -> 6
- net Net-(U1-XI): track 88.9 -> 35.1 mm
- net Net-(J2-Pin_2): track 118.1 -> 88.8 mm, vias 3 -> 2
- net Net-(J1-CC2): track 32.7 -> 12.9 mm
- net Net-(U1-UD+): track 22.4 -> 40.0 mm, vias 1 -> 2
- net Net-(U1-UD-): track 20.1 -> 33.6 mm
- net Net-(D1-K): track 12.7 -> 23.8 mm
- net Net-(J1-CC1): track 23.8 -> 17.7 mm, vias 1 -> 0
- net Net-(U1-V3): track 4.15 -> 9.75 mm
- net Net-(J2-Pin_4): track 22.0 -> 18.8 mm
- net Net-(J2-Pin_3): track 24.1 -> 22.3 mm
Other:
- board outline added: 70.2 x 64.2 mm
